File: HW/CAD/Eagle/sGPSDO_MCU_1V0.brd (EAGLE design)
At the start: 48.9 x 62.9 mm, 46 parts, among them U311 LMH6645MF, U411 LMH6645MF, U511 744059M

Commit message: HW - Eagle - sGPSDO_MCU hardware ready for the PCB house V1.0
Parts:
- moved C511 11.7 mm to (29.2, 19.1), turned to 180 degrees
- moved R558 11.4 mm to (28.6, 26.0), turned to 180 degrees
- moved R578 11.4 mm to (28.6, 26.0), turned to 180 degrees
- moved R557 10.9 mm to (28.6, 24.8), turned to 180 degrees
- moved R577 10.9 mm to (28.6, 24.8), turned to 180 degrees
- moved R555 10.9 mm to (28.6, 22.2), turned to 180 degrees
- moved R575 10.9 mm to (28.6, 22.2), turned to 180 degrees
- moved R556 10.8 mm to (28.6, 23.5), turned to 180 degrees
- moved R576 10.8 mm to (28.6, 23.5), turned to 180 degrees
- moved R554 9.67 mm to (42.5, 26.0), turned to 0 degrees
- moved R574 9.67 mm to (42.5, 26.0), turned to 0 degrees
- moved R551 9.16 mm to (42.5, 22.2), turned to 0 degrees
- moved R571 9.16 mm to (42.5, 22.2), turned to 0 degrees
- moved R553 9.16 mm to (42.5, 24.8), turned to 0 degrees
- moved R573 9.16 mm to (42.5, 24.8), turned to 0 degrees
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Routing:
- net A1_SPI1_SCK: track 0.00 -> 109.0 mm
- net D1_UBLOX_USART1_TX: track 0.00 -> 69.7 mm
- net A3_V_OCXO_ADC1_IN9: track 0.00 -> 62.2 mm
- net D0_UBLOX_USART_RX: track 0.00 -> 62.0 mm, vias 0 -> 1
- net D5_I2C1_SCL: track 0.00 -> 60.4 mm
- net D4_I2C1_SDA: track 0.00 -> 58.3 mm
- net D13_DCF77_PHASE_TIM2_CH2: track 0.00 -> 56.1 mm
- net GND: track 14.3 -> 65.6 mm, vias 3 -> 6
- net A4_V_HOLD_ADC1_IN10: track 0.00 -> 39.7 mm
- net D2_OCXO_LCKD_GPIO_O: track 0.00 -> 36.3 mm, vias 0 -> 1
- net D6_V_DCF77_DEMOD_ADC1_IN16: track 0.00 -> 36.1 mm
- net D10_PLL_LCKD_GPIO_I: track 0.00 -> 33.2 mm
- net A5_SPI1_MISO: track 0.00 -> 30.3 mm
- net D11_ONEWIRE_GPIO_IO: track 0.00 -> 28.6 mm
- net +5V: track 23.4 -> 47.9 mm, vias 4 -> 14
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Other:
- board size 48.9 x 62.9 mm -> 45.1 x 62.9 mm
- board text added: "74HC4059"
